File: Brett-RGB.sch (KiCad schematic (older format))
At the start: 141 parts, among them SW1 SW_PUSH, SW10 SW_PUSH, SW11 SW_PUSH, SW12 SW_PUSH, SW13 SW_PUSH, SW14 SW_PUSH, SW15 SW_PUSH, SW16 SW_PUSH, SW17 SW_PUSH, SW18 SW_PUSH, SW19 SW_PUSH, SW2 SW_PUSH, SW20 SW_PUSH, SW21 SW_PUSH, SW22 SW_PUSH, SW23 SW_PUSH, SW24 SW_PUSH, SW25 SW_PUSH, SW26 SW_PUSH, SW27 SW_PUSH, SW28 SW_PUSH, SW29 SW_PUSH, SW3 SW_PUSH, SW30 SW_PUSH, SW31 SW_PUSH, SW32 SW_PUSH, SW33 SW_PUSH, SW34 SW_PUSH, SW35 SW_PUSH, SW36 SW_PUSH, SW37 SW_PUSH, SW38 SW_PUSH, SW39 SW_PUSH, SW4 SW_PUSH, SW40 SW_PUSH, SW41 SW_PUSH, SW42 SW_PUSH, SW43 SW_PUSH, SW44 SW_PUSH, SW45 SW_PUSH, SW46 SW_PUSH, SW47 SW_PUSH, SW5 SW_PUSH, SW6 SW_PUSH, SW7 SW_PUSH, SW8 SW_PUSH, SW9 SW_PUSH

Commit message: Reworked the Board
Parts:
- removed D1, D10, D11, D12, D13, D14, D15, D16, D17, D18, D19, D2, D20, D21, D22, D23, D24, D25, D26, D27, D28, D29, D3, D30, D31, D32, D33, D34, D35, D36, D37, D38, D39, D4, D40, D41, D42, D43, D44, D45, D46, D47, D5, D6, D7, D8, D9: LED_RGB, mx2a:plcc-6, symbol LED_RGB
- added LED1, LED10, LED11, LED12, LED13, LED14, LED15, LED16, LED17, LED18, LED19, LED2, LED20, LED21, LED22, LED23, LED24, LED25, LED26, LED27, LED28, LED29, LED3, LED30, LED31, LED32, LED33, LED34, LED35, LED36, LED37, LED38, LED39, LED4, LED40, LED41, LED42, LED43, LED44, LED45, LED46, LED47, LED5, LED6, LED7, LED8, LED9: Led_RGB_CA, lib.pretty:RGB-0606, symbol Led_RGB_CA
- D1: renamed from D49; footprint Diodes_SMD:SOD-123 -> lib.pretty:SOD-123
- D10: renamed from D58; footprint Diodes_SMD:SOD-123 -> lib.pretty:SOD-123
- D11: renamed from D59; footprint Diodes_SMD:SOD-123 -> lib.pretty:SOD-123
- D12: renamed from D60; footprint Diodes_SMD:SOD-123 -> lib.pretty:SOD-123
- D13: renamed from D61; footprint Diodes_SMD:SOD-123 -> lib.pretty:SOD-123
- D14: renamed from D62; footprint Diodes_SMD:SOD-123 -> lib.pretty:SOD-123
- D15: renamed from D63; footprint Diodes_SMD:SOD-123 -> lib.pretty:SOD-123
- D16: renamed from D64; footprint Diodes_SMD:SOD-123 -> lib.pretty:SOD-123
- D17: renamed from D65; footprint Diodes_SMD:SOD-123 -> lib.pretty:SOD-123
- D18: renamed from D66; footprint Diodes_SMD:SOD-123 -> lib.pretty:SOD-123
- D19: renamed from D67; footprint Diodes_SMD:SOD-123 -> lib.pretty:SOD-123
- D2: renamed from D50; footprint Diodes_SMD:SOD-123 -> lib.pretty:SOD-123
- D20: renamed from D68; footprint Diodes_SMD:SOD-123 -> lib.pretty:SOD-123
- D21: renamed from D69; footprint Diodes_SMD:SOD-123 -> lib.pretty:SOD-123
- D22: renamed from D70; footprint Diodes_SMD:SOD-123 -> lib.pretty:SOD-123
- D23: renamed from D71; footprint Diodes_SMD:SOD-123 -> lib.pretty:SOD-123
- D24: renamed from D72; footprint Diodes_SMD:SOD-123 -> lib.pretty:SOD-123
- D25: renamed from D73; footprint Diodes_SMD:SOD-123 -> lib.pretty:SOD-123
- D26: renamed from D74; footprint Diodes_SMD:SOD-123 -> lib.pretty:SOD-123
- D27: renamed from D75; footprint Diodes_SMD:SOD-123 -> lib.pretty:SOD-123
- D28: renamed from D76; footprint Diodes_SMD:SOD-123 -> lib.pretty:SOD-123
- D29: renamed from D77; footprint Diodes_SMD:SOD-123 -> lib.pretty:SOD-123
- D3: renamed from D51; footprint Diodes_SMD:SOD-123 -> lib.pretty:SOD-123
- D30: renamed from D78; footprint Diodes_SMD:SOD-123 -> lib.pretty:SOD-123
- D31: renamed from D79; footprint Diodes_SMD:SOD-123 -> lib.pretty:SOD-123
- D32: renamed from D80; footprint Diodes_SMD:SOD-123 -> lib.pretty:SOD-123
- D33: renamed from D81; footprint Diodes_SMD:SOD-123 -> lib.pretty:SOD-123
- D34: renamed from D82; footprint Diodes_SMD:SOD-123 -> lib.pretty:SOD-123
- D35: renamed from D83; footprint Diodes_SMD:SOD-123 -> lib.pretty:SOD-123
- D36: renamed from D84; footprint Diodes_SMD:SOD-123 -> lib.pretty:SOD-123
- D37: renamed from D85; footprint Diodes_SMD:SOD-123 -> lib.pretty:SOD-123
- D38: renamed from D86; footprint Diodes_SMD:SOD-123 -> lib.pretty:SOD-123
- D39: renamed from D87; footprint Diodes_SMD:SOD-123 -> lib.pretty:SOD-123
- D4: renamed from D52; footprint Diodes_SMD:SOD-123 -> lib.pretty:SOD-123
- D40: renamed from D88; footprint Diodes_SMD:SOD-123 -> lib.pretty:SOD-123
- D41: renamed from D89; footprint Diodes_SMD:SOD-123 -> lib.pretty:SOD-123
- D42: renamed from D90; footprint Diodes_SMD:SOD-123 -> lib.pretty:SOD-123
- D43: renamed from D91; footprint Diodes_SMD:SOD-123 -> lib.pretty:SOD-123
- D44: renamed from D92; footprint Diodes_SMD:SOD-123 -> lib.pretty:SOD-123
- D45: renamed from D93; footprint Diodes_SMD:SOD-123 -> lib.pretty:SOD-123
- D46: renamed from D94; footprint Diodes_SMD:SOD-123 -> lib.pretty:SOD-123
- D47: renamed from D95; footprint Diodes_SMD:SOD-123 -> lib.pretty:SOD-123
- D5: renamed from D53; footprint Diodes_SMD:SOD-123 -> lib.pretty:SOD-123
- D6: renamed from D54; footprint Diodes_SMD:SOD-123 -> lib.pretty:SOD-123
- D7: renamed from D55; footprint Diodes_SMD:SOD-123 -> lib.pretty:SOD-123
- D8: renamed from D56; footprint Diodes_SMD:SOD-123 -> lib.pretty:SOD-123
- D9: renamed from D57; footprint Diodes_SMD:SOD-123 -> lib.pretty:SOD-123
- SW1, SW10, SW11, SW12, SW13, SW14, SW15, SW16, SW17, SW18, SW19, SW2, SW20, SW21, SW22, SW23, SW24, SW25, SW26, SW27, SW28, SW29, SW3, SW30, SW31, SW32, SW33, SW34, SW35, SW36, SW37, SW38, SW39, SW4, SW40, SW41, SW42, SW43, SW44, SW45, SW46, SW47, SW5, SW6, SW7, SW8, SW9: footprint mx2a:RomerG -> lib.pretty:RomerG
Connections:
- new net CS1: LED17.1, LED29.1, LED41.1, LED5.1
- new net CS10: LED14.1, LED2.1, LED26.1, LED38.1
- new net CS11: LED15.1, LED27.1, LED3.1, LED39.1
- new net CS12: LED16.1, LED28.1, LED4.1, LED40.1
- new net CS2: LED18.1, LED30.1, LED42.1, LED6.1
- new net CS3: LED19.1, LED31.1, LED7.1
- new net CS4: LED20.1, LED32.1, LED43.1, LED8.1
- new net CS5: LED21.1, LED33.1, LED44.1, LED9.1
- new net CS6: LED10.1, LED22.1, LED34.1, LED45.1
- new net CS7: LED11.1, LED23.1, LED35.1, LED46.1
- new net CS8: LED12.1, LED24.1, LED36.1, LED47.1
- new net CS9: LED1.1, LED13.1, LED25.1, LED37.1
- new net SW1: LED1.2 (R), LED10.2 (R), LED11.2 (R), LED12.2 (R), LED2.2 (R), LED3.2 (R), LED4.2 (R), LED5.2 (R), LED6.2 (R), LED7.2 (R), LED8.2 (R), LED9.2 (R)
- new net SW10: LED37.2 (R), LED38.2 (R), LED39.2 (R), LED40.2 (R), LED41.2 (R), LED42.2 (R), LED43.2 (R), LED44.2 (R), LED45.2 (R), LED46.2 (R), LED47.2 (R)
- new net SW11: LED37.3 (G), LED38.3 (G), LED39.3 (G), LED40.3 (G), LED41.3 (G), LED42.3 (G), LED43.3 (G), LED44.3 (G), LED45.3 (G), LED46.3 (G), LED47.3 (G)
- new net SW12: LED37.4 (B), LED38.4 (B), LED39.4 (B), LED40.4 (B), LED41.4 (B), LED42.4 (B), LED43.4 (B), LED44.4 (B), LED45.4 (B), LED46.4 (B), LED47.4 (B)
- new net SW2: LED1.3 (G), LED10.3 (G), LED11.3 (G), LED12.3 (G), LED2.3 (G), LED3.3 (G), LED4.3 (G), LED5.3 (G), LED6.3 (G), LED7.3 (G), LED8.3 (G), LED9.3 (G)
- new net SW3: LED1.4 (B), LED10.4 (B), LED11.4 (B), LED12.4 (B), LED2.4 (B), LED3.4 (B), LED4.4 (B), LED5.4 (B), LED6.4 (B), LED7.4 (B), LED8.4 (B), LED9.4 (B)
- new net SW4: LED13.2 (R), LED14.2 (R), LED15.2 (R), LED16.2 (R), LED17.2 (R), LED18.2 (R), LED19.2 (R), LED20.2 (R), LED21.2 (R), LED22.2 (R), LED23.2 (R), LED24.2 (R)
- new net SW5: LED13.3 (G), LED14.3 (G), LED15.3 (G), LED16.3 (G), LED17.3 (G), LED18.3 (G), LED19.3 (G), LED20.3 (G), LED21.3 (G), LED22.3 (G), LED23.3 (G), LED24.3 (G)
- new net SW6: LED13.4 (B), LED14.4 (B), LED15.4 (B), LED16.4 (B), LED17.4 (B), LED18.4 (B), LED19.4 (B), LED20.4 (B), LED21.4 (B), LED22.4 (B), LED23.4 (B), LED24.4 (B)
- new net SW7: LED25.2 (R), LED26.2 (R), LED27.2 (R), LED28.2 (R), LED29.2 (R), LED30.2 (R), LED31.2 (R), LED32.2 (R), LED33.2 (R), LED34.2 (R), LED35.2 (R), LED36.2 (R)
- new net SW8: LED25.3 (G), LED26.3 (G), LED27.3 (G), LED28.3 (G), LED29.3 (G), LED30.3 (G), LED31.3 (G), LED32.3 (G), LED33.3 (G), LED34.3 (G), LED35.3 (G), LED36.3 (G)
- new net SW9: LED25.4 (B), LED26.4 (B), LED27.4 (B), LED28.4 (B), LED29.4 (B), LED30.4 (B), LED31.4 (B), LED32.4 (B), LED33.4 (B), LED34.4 (B), LED35.4 (B), LED36.4 (B)
- no-connect marks 21 -> 0
Other:
- note removed: "Anode"
- note removed: "Cathode"
